File: submissions/klackygears/Flying_MX.kicad_pcb (KiCad board)
At the start: 2 copper layers, 88.9 x 50.8 mm, 43 parts, among them SW1 SW_Push, U1 ATmega32U4-AU, Y1 16MHz

Commit message: editing rear silk
Parts:
- moved G*** 6.02 mm to (86.4, 74.2)
- moved G*** 4.90 mm to (93.4, 61.3)
Changed lines of the file:
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@@
   )
   (module KiCadImages:FlyingMX_smallsilk (layer B.Cu)
-    (at 97.2 64.4 180)
+    (at 93.4 61.3 180)
     (fp_text reference G*** (at 0 0) (layer B.SilkS) hide
       (effects (font (size 1.524 1.524) (thickness 0.3)) (justify mirror))
@@
   )
   (module KiCadImages:FlyingMX_smallsilk (layer B.Cu)
-    (at 83.2 69.1 180)
+    (at 86.4 74.2 180)
     (fp_text reference G*** (at 0 0) (layer B.SilkS) hide
       (effects (font (size 1.524 1.524) (thickness 0.3)) (justify mirror))

Commit message: changing routing
Parts:
- removed the G*** at (93.4, 61.3)
- removed the G*** at (54.6, 41.5)
- removed the G*** at (133.3, 46.6)
- removed the G*** at (86.4, 74.2)
- removed the G*** at (112.2, 70.9)
- removed the G*** at (75.6, 43.4)
- removed the G*** at (101.0, 42.5)
- removed the G*** at (55.3, 58.5)
- added G***: LOGO, KiCadImages:FlyingMX_largesilk, B.Cu at (59.7, 65.2)
- added G***: LOGO, KiCadImages:FlyingMX_medsilk, B.Cu at (72.4, 45.2)
- added G***: LOGO, KiCadImages:FlyingMX_smallsilk, B.Cu at (106.6, 32.7)
- added G***: LOGO, KiCadImages:FlyingMX_smallsilk, B.Cu at (131.6, 67.6)
- added G***: LOGO, KiCadImages:FlyingMX_largesilk, B.Cu at (121.0, 47.6)
- added G***: LOGO, KiCadImages:FlyingMX_smallsilk, B.Cu at (55.8, 34.8)
- added G***: LOGO, KiCadImages:FlyingMX_smallsilk, B.Cu at (93.3, 60.7)
- added G***: LOGO, KiCadImages:FlyingMX_medsilk, B.Cu at (112.3, 72.1)
- added G***: LOGO, KiCadImages:FlyingMX_medsilk, B.Cu at (89.0, 38.4)
- moved C1 43.1 mm to (113.5, 68.2), turned to 180 degrees
- moved Y1 36.9 mm to (113.5, 63.8), turned to 90 degrees
- moved C2 30.7 mm to (113.5, 59.4), turned to 0 degrees
- moved D7 22.0 mm to (95.3, 33.6), turned to 225 degrees
- moved D4 16.3 mm to (85.8, 37.6), turned to 225 degrees
- moved D6 14.6 mm to (80.3, 33.6), turned to 225 degrees
- moved D3 9.05 mm to (70.8, 37.6), turned to 225 degrees
- moved D5 7.35 mm to (65.3, 33.6), turned to 225 degrees
- moved SW1 2.89 mm to (109.6, 34.8), turned to 0 degrees
- moved D2 2.61 mm to (55.8, 37.6), turned to 225 degrees
- moved G*** 0.10 mm to (134.1, 34.9)
Connections:
- U1 pad 18: ROW1 -> Net-(U1-Pad18)
- U1 pad 19: ROW0 -> Net-(U1-Pad19)
- U1 pad 26: Net-(U1-Pad26) -> ROW1
- U1 pad 27: Net-(U1-Pad27) -> ROW0
- U1 pad 28: COL2 -> COL0
- U1 pad 30: COL0 -> COL2
Routing:
- net GND: track 301.0 -> 224.5 mm, vias 6 -> 2
- net Net-(C1-Pad1): track 51.9 -> 10.6 mm
- net Net-(C2-Pad1): track 47.4 -> 11.0 mm
- net Net-(D4-Pad2): track 34.1 -> 18.0 mm, vias 1 -> 0
- net ROW1: track 85.8 -> 100.5 mm, vias 3 -> 0
- net VCC: track 186.6 -> 173.6 mm, vias 5 -> 3
- net Net-(D6-Pad2): track 37.8 -> 47.8 mm
- net ROW0: track 86.7 -> 78.7 mm, vias 4 -> 0
- net Net-(D5-Pad2): track 38.2 -> 46.0 mm
- net Net-(D3-Pad2): track 21.9 -> 14.8 mm, vias 1 -> 0
- net Net-(R1-Pad2): track 25.7 -> 32.6 mm
- net COL2: track 80.6 -> 87.4 mm, vias 2 -> 1
- net Net-(D2-Pad2): track 19.8 -> 13.1 mm, vias 1 -> 0
- net +5V: track 124.8 -> 130.2 mm, vias 6 -> 4
- net Net-(D10-Pad3): track 42.4 -> 38.1 mm
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- added copper zone on B.Cu, net GND
