File: submissions/klackygears/Flying_MX.kicad_pcb (KiCad board)
At the start: 2 copper layers, 88.9 x 50.8 mm, 47 parts, among them J1 USB_C_Receptacle, SW1 SW_Push, U1 ATmega32U4-AU, U2 PRTR5V0U2X, Y1 16MHz

Commit message: moving things around a bit
Parts:
- moved G*** 1.03 mm to (115.5, 42.5)
Changed lines of the file:
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@@
   )
   (module KiCadImages:GearLogo_smallsolder (layer F.Cu)
-    (at 115 41.6)
+    (at 115.5 42.5)
     (fp_text reference G*** (at 0 0) (layer F.SilkS) hide
       (effects (font (size 1.524 1.524) (thickness 0.3)))

Commit message: correcting & improving some things
Parts:
- removed the G*** at (115.5, 42.5)
- removed the G*** at (68.6, 59.8)
- removed the G*** at (59.9, 40.7)
- removed the G*** at (91.4, 60.4)
- removed the G*** at (90.0, 51.9)
- removed the G*** at (133.8, 71.8)
- removed the G*** at (114.5, 71.4)
- removed the G*** at (122.5, 50.3)
- removed the G*** at (79.8, 38.4)
- removed the G*** at (96.5, 35.9)
- added G***: LOGO, KiCadImages:GearLogo_smallsolder, B.Cu at (114.7, 43.1)
- added G***: LOGO, KiCadImages:FlyingMX_largesilk, B.Cu at (63.9, 61.3)
- added G***: LOGO, KiCadImages:GearLogo_smallsolder, F.Cu at (114.7, 43.2)
- added G***: LOGO, KiCadImages:FlyingMX_smallsilk, B.Cu at (55.0, 35.0)
- added G***: LOGO, KiCadImages:FlyingMX_smallsilk, B.Cu at (90.5, 41.9)
- added G***: LOGO, KiCadImages:FlyingMX_smallsilk, B.Cu at (110.1, 68.4)
- added G***: LOGO, KiCadImages:FlyingMX_smallsilk, B.Cu at (98.0, 36.0)
- added G***: LOGO, KiCadImages:FlyingMX_smallsilk, B.Cu at (133.2, 75.1)
- added G***: LOGO, KiCadImages:FlyingMX_medsilk, B.Cu at (89.6, 60.3)
- added G***: LOGO, KiCadImages:FlyingMX_medsilk, B.Cu at (70.6, 37.8)
- added G***: LOGO, KiCadImages:FlyingMX_largesilk, B.Cu at (122.0, 53.0)
- J1: value USB_C_Receptacle -> USB_C_Receptacle_USB2.0
- moved J1 1.20 mm to (126.5, 35.9)
Routing:
- net Net-(R1-Pad2): track 32.6 -> 34.8 mm
- net VCC: track 189.4 -> 191.1 mm
- net D+: track 18.6 -> 17.2 mm
- net Net-(J1-PadB5): track 12.7 -> 14.0 mm
- net Net-(J1-PadA5): track 9.74 -> 10.5 mm
