File: submissions/klackygears/Flying_MX.kicad_pcb (KiCad board)
At the start: 2 copper layers, 88.9 x 50.8 mm, 48 parts, among them J1 USB_C_Receptacle_USB2.0, SW1 SW_Push, U1 ATmega32U4-AU, U2 PRTR5V0U2X, Y1 16MHz

Commit message: updating footprints and silk
Parts:
- removed the G*** at (114.7, 43.1)
- removed the G*** at (63.9, 61.3)
- removed the G*** at (114.7, 43.2)
- removed the G*** at (55.0, 35.0)
- removed the G*** at (90.5, 41.9)
- removed the G*** at (110.1, 68.4)
- removed the G*** at (98.0, 36.0)
- removed the G*** at (133.2, 75.1)
- removed the G*** at (89.6, 60.3)
- removed the G*** at (70.6, 37.8)
- removed the G*** at (122.0, 53.0)
- added G***: LOGO, Flying_MX:GearLogo_smallsolder, F.Cu at (114.8, 42.5)
- added G***: LOGO, Flying_MX:FlyingMX_medsilk, B.Cu at (91.1, 55.2)
- added G***: LOGO, Flying_MX:FlyingMX_medsilk, B.Cu at (64.5, 37.3)
- added G***: LOGO, Flying_MX:FlyingMX_largesilk, B.Cu at (120.6, 52.0)
- added G***: LOGO, Flying_MX:FlyingMX_largesilk, B.Cu at (67.4, 60.9)
- added G***: LOGO, Flying_MX:GearLogo_smallsolder, B.Cu at (133.7, 75.6)
- added G***: LOGO, Flying_MX:FlyingMX_smallsilk, B.Cu at (90.1, 72.2)
- added G***: LOGO, Flying_MX:FlyingMX_smallsilk, B.Cu at (53.7, 34.6)
- added G***: LOGO, Flying_MX:FlyingMX_smallsilk, B.Cu at (109.9, 65.7)
- added G***: LOGO, Flying_MX:FlyingMX_smallsilk, B.Cu at (114.3, 74.6)
- added G***: LOGO, Flying_MX:FlyingMX_smallsilk, B.Cu at (86.4, 41.2)
- added G***: LOGO, Flying_MX:FlyingMX_smallsilk, B.Cu at (112.0, 35.0)
- added G***: LOGO, Flying_MX:FlyingMX_medsilk, B.Cu at (100.8, 42.1)
- D10, D11, D12, D13, D8, D9: footprint KiCadLibs:SK6812MINI-E -> Flying_MX:SK6812MINI-E
- MX1, MX2, MX3, MX4, MX5, MX6: footprint Universal-Switch-Footprint:MX-ALPs-PG1350-FLIP -> Flying_MX:MX-ALPs-PG1350-FLIP
- SW1: footprint random-keyboard-parts:SKQG-1155865 -> Flying_MX:SKQG-1155865
- U2: footprint random-keyboard-parts:SOT143B -> Flying_MX:SOT143B
