File: submissions/Kyrremann/kyrremann.sch (KiCad schematic (older format))
At the start: 38 parts, among them J1 USB_C_Receptacle_USB2.0, J2 Conn_01x06_Female, J3 Conn_01x06_Female, SW1 SW_Push, U1 ATmega32U2-MU, Y1 16Mhz

Commit message: Retraced the keyboard, and added cool silks
Parts:
- C1, C2, C3: LCSC (none) -> C15849
- C4: LCSC (none) -> C14663
- D1, D10, D2, D3, D4, D5, D6, D7, D8, D9: LCSC (none) -> C81598
- R1, R2: LCSC (none) -> C23186
- R3, R4: LCSC (none) -> C23345
- R5, R6: LCSC (none) -> C25804
- U1: LCSC (none) -> C57345
- Y1: footprint Crystal:Crystal_SMD_3225-4Pin_3.2x2.5mm_HandSoldering -> Crystal:Crystal_SMD_3225-4Pin_3.2x2.5mm; LCSC (none) -> C13738
Connections:
- net GND: no longer J1.S1 (SHIELD)
- no-connect marks 15 -> 16
Changed lines of the file:
@@
 F 2 "Package_DFN_QFN:QFN-32-1EP_5x5mm_P0.5mm_EP3.1x3.1mm" H 4550 3200 50  0001 C CIN
 F 3 "http://ww1.microchip.com/downloads/en/DeviceDoc/doc7799.pdf" H 4550 3200 50  0001 C CNN
+F 4 "C57345" H 4550 3200 50  0001 C CNN "LCSC"
 	1    4550 3200
 	1    0    0    -1
@@
 F 2 "Resistor_SMD:R_0603_1608Metric_Pad1.05x0.95mm_HandSolder" V 2180 3050 50  0001 C CNN
 F 3 "~" H 2250 3050 50  0001 C CNN
+F 4 "C23186" H 2250 3050 50  0001 C CNN "LCSC"
 	1    2250 3050
 	0    1    1    0
@@
 F 2 "Resistor_SMD:R_0603_1608Metric_Pad1.05x0.95mm_HandSolder" V 2180 3150 50  0001 C CNN
 F 3 "~" H 2250 3150 50  0001 C CNN
+F 4 "C23186" H 2250 3150 50  0001 C CNN "LCSC"
 	1    2250 3150
 	0    -1   -1   0
@@
 L power:GND #PWR010
 U 1 1 5E98FED8
-P 1100 4450
-F 0 "#PWR010" H 1100 4200 50  0001 C CNN
-F 1 "GND" H 1105 4277 50  0000 C CNN
-F 2 "" H 1100 4450 50  0001 C CNN
-F 3 "" H 1100 4450 50  0001 C CNN
-	1    1100 4450
-	1    0    0    -1
-$EndComp
-Wire Wire Line
-	950  4350 950  4450
-Wire Wire Line
-	950  4450 1100 4450
-Wire Wire Line
-	1100 4450 1250 4450
-Wire Wire Line
-	1250 4450 1250 4350
-Connection ~ 1100 4450
+P 1250 4350
+F 0 "#PWR010" H 1250 4100 50  0001 C CNN
+F 1 "GND" H 1255 4177 50  0000 C CNN
+F 2 "" H 1250 4350 50  0001 C CNN
+F 3 "" H 1250 4350 50  0001 C CNN
+	1    1250 4350
+	1    0    0    -1
+$EndComp
 NoConn ~ 1850 3950
 NoConn ~ 1850 4050
@@
 F 2 "Resistor_SMD:R_0603_1608Metric_Pad1.05x0.95mm_HandSolder" V 3530 2700 50  0001 C CNN
 F 3 "~" H 3600 2700 50  0001 C CNN
+F 4 "C23345" H 3600 2700 50  0001 C CNN "LCSC"
 	1    3600 2700
 	0    1    1    0
@@
 F 2 "Resistor_SMD:R_0603_1608Metric_Pad1.05x0.95mm_HandSolder" V 3530 2800 50  0001 C CNN
 F 3 "~" H 3600 2800 50  0001 C CNN
+F 4 "C23345" H 3600 2800 50  0001 C CNN "LCSC"
 	1    3600 2800
 	0    -1   -1   0
@@
 F 2 "Resistor_SMD:R_0603_1608Metric_Pad1.05x0.95mm_HandSolder" V 5530 4300 50  0001 C CNN
 F 3 "~" H 5600 4300 50  0001 C CNN
+F 4 "C25804" H 5600 4300 50  0001 C CNN "LCSC"
 	1    5600 4300
 	0    1    1    0
@@
 F 2 "Resistor_SMD:R_0603_1608Metric_Pad1.05x0.95mm_HandSolder" V 5580 1450 50  0001 C CNN
 F 3 "~" H 5650 1450 50  0001 C CNN
+F 4 "C25804" H 5650 1450 50  0001 C CNN "LCSC"
 	1    5650 1450
 	1    0    0    -1
@@
 F 2 "Capacitor_SMD:C_0603_1608Metric_Pad1.05x0.95mm_HandSolder" H 1538 1500 50  0001 C CNN
 F 3 "~" H 1500 1650 50  0001 C CNN
+F 4 "C15849" H 1500 1650 50  0001 C CNN "LCSC"
 	1    1500 1650
 	1    0    0    -1
@@
 F 2 "Capacitor_SMD:C_0603_1608Metric_Pad1.05x0.95mm_HandSolder" H 1888 1500 50  0001 C CNN
 F 3 "~" H 1850 1650 50  0001 C CNN
+F 4 "C15849" H 1850 1650 50  0001 C CNN "LCSC"
 	1    1850 1650
 	1    0    0    -1
@@
 F 2 "Capacitor_SMD:C_0603_1608Metric_Pad1.05x0.95mm_HandSolder" H 2238 1500 50  0001 C CNN
 F 3 "~" H 2200 1650 50  0001 C CNN
+F 4 "C14663" H 2200 1650 50  0001 C CNN "LCSC"
 	1    2200 1650
 	1    0    0    -1
@@
 F 2 "Capacitor_SMD:C_0603_1608Metric_Pad1.05x0.95mm_HandSolder" H 2688 1500 50  0001 C CNN
 F 3 "~" H 2650 1650 50  0001 C CNN
+F 4 "C15849" H 2650 1650 50  0001 C CNN "LCSC"
 	1    2650 1650
 	1    0    0    -1
@@
 F 0 "Y1" H 2894 4346 50  0000 L CNN
 F 1 "16Mhz" H 2900 4450 50  0000 L CNN
-F 2 "Crystal:Crystal_SMD_3225-4Pin_3.2x2.5mm_HandSoldering" H 2700 4300 50  0001 C CNN
+F 2 "Crystal:Crystal_SMD_3225-4Pin_3.2x2.5mm" H 2700 4300 50  0001 C CNN
 F 3 "~" H 2700 4300 50  0001 C CNN
+F 4 "C13738" H 2700 4300 50  0001 C CNN "LCSC"
 	1    2700 4300
 	1    0    0    -1
@@
 F 2 "Diode_SMD:D_SOD-123" H 7150 2200 50  0001 C CNN
 F 3 "~" H 7150 2200 50  0001 C CNN
+F 4 "C81598" H 7150 2200 50  0001 C CNN "LCSC"
 	1    7150 2200
 	0    -1   -1   0
@@
 F 2 "Diode_SMD:D_SOD-123" H 7450 2200 50  0001 C CNN
 F 3 "~" H 7450 2200 50  0001 C CNN
+F 4 "C81598" H 7450 2200 50  0001 C CNN "LCSC"
 	1    7450 2200
 	0    -1   -1   0
@@
 F 2 "Diode_SMD:D_SOD-123" H 7750 2200 50  0001 C CNN
 F 3 "~" H 7750 2200 50  0001 C CNN
+F 4 "C81598" H 7750 2200 50  0001 C CNN "LCSC"
 	1    7750 2200
 	0    -1   -1   0
@@
 F 2 "Diode_SMD:D_SOD-123" H 8050 2200 50  0001 C CNN
 F 3 "~" H 8050 2200 50  0001 C CNN
+F 4 "C81598" H 8050 2200 50  0001 C CNN "LCSC"
 	1    8050 2200
 	0    -1   -1   0
@@
 F 2 "Diode_SMD:D_SOD-123" H 8350 2200 50  0001 C CNN
 F 3 "~" H 8350 2200 50  0001 C CNN
+F 4 "C81598" H 8350 2200 50  0001 C CNN "LCSC"
 	1    8350 2200
 	0    -1   -1   0
@@
 F 2 "Diode_SMD:D_SOD-123" H 8350 2950 50  0001 C CNN
 F 3 "~" H 8350 2950 50  0001 C CNN
+F 4 "C81598" H 8350 2950 50  0001 C CNN "LCSC"
 	1    8350 2950
 	0    -1   -1   0
@@
 F 2 "Diode_SMD:D_SOD-123" H 8050 2950 50  0001 C CNN
 F 3 "~" H 8050 2950 50  0001 C CNN
+F 4 "C81598" H 8050 2950 50  0001 C CNN "LCSC"
 	1    8050 2950
 	0    -1   -1   0
@@
 F 2 "Diode_SMD:D_SOD-123" H 7750 2950 50  0001 C CNN
 F 3 "~" H 7750 2950 50  0001 C CNN
+F 4 "C81598" H 7750 2950 50  0001 C CNN "LCSC"
 	1    7750 2950
 	0    -1   -1   0
@@
 F 2 "Diode_SMD:D_SOD-123" H 7450 2950 50  0001 C CNN
 F 3 "~" H 7450 2950 50  0001 C CNN
+F 4 "C81598" H 7450 2950 50  0001 C CNN "LCSC"
 	1    7450 2950
 	0    -1   -1   0
@@
 F 2 "Diode_SMD:D_SOD-123" H 7150 2950 50  0001 C CNN
 F 3 "~" H 7150 2950 50  0001 C CNN
+F 4 "C81598" H 7150 2950 50  0001 C CNN "LCSC"
 	1    7150 2950
 	0    -1   -1   0
@@
 NoConn ~ 5250 2700
 NoConn ~ 5250 2600
+NoConn ~ 950  4350
 $EndSCHEMATC
