File: submissions/crokto/crokto.kicad_pcb (KiCad board)
At the start: 2 copper layers, 100 x 50 mm, 156 parts, among them J1 AVR-ISP-6, K1 esc, K10 #4, K11 #5, K12 #6, K13 #7, K14 #8, K15 #9, K16 #0, K17 bsls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

Commit message: fixed footprints, added jlcpcba
Parts:
- added H3: jlc, crokto:jlc, F.Cu at (76.4, 5.10)
- added H4: jlc, crokto:JLCPCBA, F.Cu at (98.9, 1.10)
- added H5: jlc, crokto:JLCPCBA, F.Cu at (1.00, 1.00)
- added H6: jlc, crokto:JLCPCBA, F.Cu at (2.10, 49.0)
- J1: footprint crokto:2x3-jumper -> crokto2:2x3-jumper
