File: submissions/JSmurf/ASETNIOP BC.kicad_pcb (KiCad board)
At the start: 2 copper layers, 100 x 50 mm, 36 parts, among them SW1 SW_Push, U1 ATmega32U4-AU, Y1 16MHz

Commit message: Final Submission
Made some changes to the routing, added some ground fills, and added some decorative slkscreen.
Parts:
- added G***: LOGO, Kicad Silks:Silk Test Four, B.Cu at (182.0, 94.0)
- moved C5 6.00 mm to (152.8, 105.6)
- moved R4 6.00 mm to (156.8, 105.6)
Routing:
- net +5V: track 140.6 -> 152.6 mm
- net GND: track 142.9 -> 154.9 mm
- net Net-(R4-Pad2): track 32.6 -> 38.6 mm
- net COL2: track 45.2 -> 40.2 mm
- added copper zone on B.Cu, net GND
- added copper zone on F.Cu, net GND
Other:
- outline, holes or cut-outs redrawn
- board text added: "ADD"
- board text added: "Alex Cooper AlexCooperDev.com"
- board text added: "CAN"
- board text added: "IF"
- board text added: "It doesn’t fit in a rolodex Because it doesn’t belong in a rolodex"
- board text added: "NEED"
- board text added: "READ"
- board text added: "SWITCHES"
- board text added: "THIS"
- board text added: "TO"
- board text added: "YOU"
